File: psvsd/psvsd-v10.sch (EAGLE design)
At the start: 28 parts, among them J1 TRANSFLASH-PUSH, U1 USB2244QFN, Y1 24.000MHz

Commit message: DRC fixes
Parts:
- JP1: value (none) -> UART_KERMIT
- JP2: value (none) -> UART_SYSCON
- U3: value (none) -> VREG
Connections:
- net GND: now also J1.S@1, J1.S@2, J1.S@3, J1.S@4, U1.SD_WP
Changed lines of the file:
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@@
 <part name="J1" library="sd-mmc" deviceset="TRANSFLASH" device="-PUSH"/>
 <part name="U1" library="microchip" deviceset="USB2244" device="QFN"/>
-<part name="JP1" library="pinhead" deviceset="PINHD-1X5" device=""/>
-<part name="JP2" library="pinhead" deviceset="PINHD-1X5" device=""/>
-<part name="U3" library="v-reg-micrel" deviceset="MIC5219XX" device=""/>
+<part name="JP1" library="pinhead" deviceset="PINHD-1X5" device="" value="UART_KERMIT"/>
+<part name="JP2" library="pinhead" deviceset="PINHD-1X5" device="" value="UART_SYSCON"/>
+<part name="U3" library="v-reg-micrel" deviceset="MIC5219XX" device="" value="VREG"/>
 <part name="C1" library="rcl" deviceset="C-EU" device="C0603" value="1uF"/>
 <part name="GND1" library="supply1" deviceset="GND" device=""/>
@@
 <part name="C3" library="rcl" deviceset="C-EU" device="C0402" value="18pF"/>
 <part name="C4" library="rcl" deviceset="C-EU" device="C0402" value="18pF"/>
-<part name="GND3" library="supply1" deviceset="GND" device=""/>
 <part name="FB1" library="inductors" deviceset="BLM15H" device="" technology="B121SN1" value=""/>
 <part name="C5" library="rcl" deviceset="C-EU" device="C0603" value="1.0uF"/>
@@
 <part name="C15" library="rcl" deviceset="C-EU" device="C0402" value="0.1uF"/>
 <part name="GND2" library="supply1" deviceset="GND" device=""/>
+<part name="GND13" library="supply1" deviceset="GND" device=""/>
+<part name="GND3" library="supply1" deviceset="GND" device=""/>
+<part name="GND14" library="supply1" deviceset="GND" device=""/>
 </parts>
 <sheets>
@@
 <instance part="C3" gate="G$1" x="-165.1" y="-43.18"/>
 <instance part="C4" gate="G$1" x="-165.1" y="-53.34"/>
-<instance part="GND3" gate="1" x="-171.704" y="-49.276" rot="R270"/>
 <instance part="FB1" gate="G$1" x="-45.72" y="-33.02" rot="R90"/>
 <instance part="C5" gate="G$1" x="-45.72" y="-48.26"/>
@@
 <instance part="C15" gate="G$1" x="-88.9" y="-48.26"/>
 <instance part="GND2" gate="1" x="-88.9" y="-63.5"/>
+<instance part="GND13" gate="1" x="-93.98" y="-5.08"/>
+<instance part="GND3" gate="1" x="-170.18" y="-48.26" rot="R270"/>
+<instance part="GND14" gate="1" x="-60.96" y="-35.56"/>
 </instances>
 <busses>
@@
 </segment>
 <segment>
-<pinref part="GND3" gate="1" pin="GND"/>
-<pinref part="C4" gate="G$1" pin="1"/>
-<wire x1="-169.164" y1="-49.276" x2="-165.1" y2="-49.276" width="0.1524" layer="91"/>
-<wire x1="-165.1" y1="-49.276" x2="-165.1" y2="-49.53" width="0.1524" layer="91"/>
-<pinref part="C3" gate="G$1" pin="2"/>
-<wire x1="-165.1" y1="-49.53" x2="-165.1" y2="-50.8" width="0.1524" layer="91"/>
-<wire x1="-165.1" y1="-48.26" x2="-165.1" y2="-49.276" width="0.1524" layer="91"/>
-<junction x="-165.1" y="-49.53"/>
-</segment>
-<segment>
 <pinref part="C5" gate="G$1" pin="2"/>
 <pinref part="GND4" gate="1" pin="GND"/>
@@
 <wire x1="66.04" y1="17.78" x2="55.88" y2="17.78" width="0.1524" layer="91"/>
 <label x="55.88" y="17.78" size="1.778" layer="95"/>
+</segment>
+<segment>
+<pinref part="U1" gate="G$1" pin="SD_WP"/>
+<wire x1="-119.38" y1="-2.54" x2="-93.98" y2="-2.54" width="0.1524" layer="91"/>
+<pinref part="GND13" gate="1" pin="GND"/>
+</segment>
+<segment>
+<pinref part="C4" gate="G$1" pin="1"/>
+<pinref part="C3" gate="G$1" pin="2"/>
+<wire x1="-165.1" y1="-48.26" x2="-165.1" y2="-50.8" width="0.1524" layer="91"/>
+<wire x1="-165.1" y1="-48.26" x2="-167.64" y2="-48.26" width="0.1524" layer="91"/>
+<junction x="-165.1" y="-48.26"/>
+<pinref part="GND3" gate="1" pin="GND"/>
+</segment>
+<segment>
+<pinref part="J1" gate="G$1" pin="S@1"/>
+<wire x1="-63.5" y1="-20.32" x2="-60.96" y2="-20.32" width="0.1524" layer="91"/>
+<wire x1="-60.96" y1="-20.32" x2="-60.96" y2="-22.86" width="0.1524" layer="91"/>
+<pinref part="J1" gate="G$1" pin="S@2"/>
+<wire x1="-60.96" y1="-22.86" x2="-60.96" y2="-25.4" width="0.1524" layer="91"/>
+<wire x1="-60.96" y1="-25.4" x2="-60.96" y2="-27.94" width="0.1524" layer="91"/>
+<wire x1="-60.96" y1="-27.94" x2="-60.96" y2="-33.02" width="0.1524" layer="91"/>
+<wire x1="-63.5" y1="-22.86" x2="-60.96" y2="-22.86" width="0.1524" layer="91"/>
+<junction x="-60.96" y="-22.86"/>
+<pinref part="J1" gate="G$1" pin="S@3"/>
+<wire x1="-63.5" y1="-25.4" x2="-60.96" y2="-25.4" width="0.1524" layer="91"/>
+<junction x="-60.96" y="-25.4"/>
+<pinref part="J1" gate="G$1" pin="S@4"/>
+<wire x1="-63.5" y1="-27.94" x2="-60.96" y2="-27.94" width="0.1524" layer="91"/>
+<junction x="-60.96" y="-27.94"/>
+<pinref part="GND14" gate="1" pin="GND"/>
 </segment>
 </net>
@@
 <wire x1="-170.18" y1="35.56" x2="-177.8" y2="35.56" width="0.1524" layer="91"/>
 <junction x="-177.8" y="35.56"/>
-</segment>
-<segment>
+<junction x="-177.8" y="40.64"/>
+</segment>
+<segment>

Commit message: More cleanups
Parts:
- U1: device microchip:USB2244QFN -> USB2244:USB2244QFN
Connections:
- net CRD_PWR renamed VDD
