File: psvsd/psvsd-v20.brd (EAGLE design)
At the start: 30 x 33.2 mm, 26 parts, among them U1 GL823(A)OG, U2 74AUP1G74DC, U3 LP3996_DSC_10

Commit message: Added USB trace clearance recommendations from GL823 design docs
Connections:
- net GND: no longer U$1.22
Routing:
- net GND: track 15.5 -> 21.1 mm
Changed lines of the file:
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@@
 <?xml version="1.0" encoding="utf-8"?>
 <!DOCTYPE eagle SYSTEM "eagle.dtd">
-<eagle version="8.2.0">
+<eagle version="8.2.2">
 <drawing>
 <settings>
@@
 <setting verticaltext="up"/>
 </settings>
-<grid distance="1" unitdist="mil" unit="mil" style="lines" multiple="1" display="yes" altdistance="0.5" altunitdist="mm" altunit="mm"/>
+<grid distance="1" unitdist="mm" unit="mm" style="lines" multiple="1" display="yes" altdistance="0.5" altunitdist="mm" altunit="mm"/>
 <layers>
 <layer number="1" name="Top" color="4" fill="1" visible="yes" active="yes"/>
@@
 <layer number="168" name="4mmHeightArea" color="7" fill="1" visible="no" active="yes"/>
 <layer number="199" name="Contour" color="7" fill="1" visible="no" active="yes"/>
-<layer number="200" name="200bmp" color="1" fill="10" visible="yes" active="yes"/>
+<layer number="200" name="200bmp" color="1" fill="10" visible="no" active="yes"/>
 <layer number="201" name="201bmp" color="2" fill="1" visible="no" active="no"/>
 <layer number="202" name="202bmp" color="3" fill="1" visible="no" active="no"/>
@@
 <class number="0" name="default" width="0" drill="0">
 </class>
+<class number="1" name="USB" width="0" drill="0">
+</class>
+<class number="2" name="Clock/HS" width="0" drill="0">
+<clearance class="1" value="1.27"/>
+</class>
+<class number="3" name="GND" width="0" drill="0">
+<clearance class="1" value="0.508"/>
+</class>
 </classes>
 <designrules name="SparkFun *">
@@
 <element name="SD1" library="Seeed-Connector" library_urn="urn:adsk.eagle:library:478" package="MICRO-SD9+4P-SMD-16.1X14.5X1.85MM" value="ST-TF-003A" x="15.05" y="16.56" smashed="yes" rot="R90">
 <attribute name="MPN" value="ST-TF-003A" x="15.05" y="16.56" size="1.778" layer="27" rot="R90" display="off"/>
+<attribute name="NAME" x="12.891" y="21.386" size="0.254" layer="33" ratio="10" rot="R90"/>
 <attribute name="NAME" x="9.9" y="30.303" size="0.6096" layer="25" ratio="11" rot="SR180"/>
-<attribute name="NAME" x="12.891" y="21.386" size="0.254" layer="33" ratio="10" rot="R90"/>
 <attribute name="VALUE" x="18.86" y="19.735" size="0.508" layer="27" ratio="10" rot="SR180"/>
 </element>
@@
 </elements>
 <signals>
-<signal name="GND">
+<signal name="GND" class="3">
 <contactref element="U$1" pad="4"/>
 <contactref element="U$1" pad="6"/>
@@
 <wire x1="20.08671875" y1="22.65" x2="21.9664" y2="20.77031875" width="0.254" layer="16"/>
 <polygon width="0.254" layer="1" rank="2">
-<vertex x="0" y="0"/>
-<vertex x="30" y="0"/>
+<vertex x="0" y="2.5"/>
+<vertex x="30" y="2.5"/>
 <vertex x="30" y="33.5"/>
 <vertex x="0" y="33.5"/>
 </polygon>
 <polygon width="0.254" layer="16">
-<vertex x="0" y="0"/>
+<vertex x="0" y="2.5"/>
 <vertex x="0" y="33.5"/>
 <vertex x="30" y="33.5"/>
-<vertex x="30" y="0"/>
+<vertex x="30" y="2.5"/>
 </polygon>
 <wire x1="15.13" y1="23.15" x2="15.88" y2="23.15" width="0.254" layer="16"/>
@@
 <via x="19.5" y="15" extent="1-16" drill="0.35"/>
 <via x="13" y="4" extent="1-16" drill="0.35"/>
-<contactref element="U$1" pad="22"/>
 <contactref element="U$1" pad="24"/>
 <contactref element="U$1" pad="34"/>
 <via x="23.5" y="22" extent="1-16" drill="0.35"/>
+<wire x1="3.226" y1="1.35" x2="3.226" y2="3.774" width="0.254" layer="1"/>
+<wire x1="3.226" y1="3.774" x2="3" y2="4" width="0.254" layer="1"/>
+<wire x1="5.626" y1="1.35" x2="5.626" y2="3.626" width="0.254" layer="1"/>
+<wire x1="5.626" y1="3.626" x2="6" y2="4" width="0.254" layer="1"/>
 </signal>
 <signal name="UART_KERMIT_RFR">
@@
 <wire x1="26.98" y1="4" x2="28.81" y2="6.33" width="0.254" layer="16"/>
 <polygon width="0.254" layer="1">
-<vertex x="19" y="0"/>
-<vertex x="30" y="0"/>
+<vertex x="19" y="2.5"/>
+<vertex x="30" y="2.5"/>
 <vertex x="30" y="10"/>
 <vertex x="19" y="10"/>
@@
 <wire x1="26.74" y1="7.63" x2="28.81" y2="7.63" width="0.254" layer="16"/>
 </signal>
-<signal name="USB_N">
+<signal name="USB_N" class="1">
 <contactref element="U$1" pad="3"/>
 <contactref element="U1" pad="3"/>
@@
 <wire x1="13.2286" y1="26.2286" x2="14" y2="27" width="0.254" layer="1"/>
 </signal>
-<signal name="USB_P">
+<signal name="USB_P" class="1">
 <contactref element="U$1" pad="5"/>
 <contactref element="U1" pad="4"/>
@@
 <wire x1="17.88" y1="26.09" x2="17.05" y2="26.92" width="0.254" layer="16"/>
 </signal>
-<signal name="SD_CLK">
+<signal name="SD_CLK" class="2">
 <contactref element="U1" pad="12"/>
 <contactref element="SD1" pad="5"/>
@@
 <wire x1="15" y1="18" x2="15" y2="16.56" width="0.254" layer="1"/>
 </signal>
-<signal name="SD_D0">
+<signal name="SD_D0" class="2">
 <contactref element="U1" pad="11"/>
 <contactref element="SD1" pad="7"/>
@@
 <wire x1="19.4" y1="17.9" x2="19.4" y2="16.56" width="0.254" layer="1"/>
 </signal>
-<signal name="SD_D1">
+<signal name="SD_D1" class="3">
 <contactref element="U1" pad="10"/>
 <contactref element="SD1" pad="8"/>
@@
 <wire x1="20.5" y1="17.75" x2="20.5" y2="16.56" width="0.254" layer="1"/>
 </signal>
-<signal name="SD_D2">
+<signal name="SD_D2" class="2">
 <contactref element="U1" pad="19"/>
 <contactref element="SD1" pad="1"/>
@@
 <wire x1="12.5" y1="16.86" x2="12.8" y2="16.56" width="0.254" layer="1"/>
 </signal>
-<signal name="SD_D3">
+<signal name="SD_D3" class="2">
 <contactref element="U1" pad="18"/>
 <contactref element="SD1" pad="2"/>

Commit message: Changed bypass value for DVDD2 and added a new ferrite bead to AVDD
Parts:
- added FB2: (no value), inductors:0402
- C3: value 0.1uF -> 10uF
- C8: value ? -> 0.1uF
- moved C6 2.69 mm to (22.2, 26.5)
Connections:
- new net AVDD: FB2.2, U1.6
- net VDD33: now also FB2.1; no longer U1.6
Routing:
- net AVDD: track 0.00 -> 1.71 mm
- net VDD33: track 57.2 -> 56.2 mm
Changed lines of the file:
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@@
 <?xml version="1.0" encoding="utf-8"?>
 <!DOCTYPE eagle SYSTEM "eagle.dtd">
-<eagle version="8.2.2">
+<eagle version="8.2.0">
 <drawing>
 <settings>
@@
 <layers>
 <layer number="1" name="Top" color="4" fill="1" visible="yes" active="yes"/>
+<layer number="2" name="Route2" color="1" fill="3" visible="no" active="no"/>
+<layer number="3" name="Route3" color="4" fill="3" visible="no" active="no"/>
+<layer number="4" name="Route4" color="1" fill="4" visible="no" active="no"/>
+<layer number="5" name="Route5" color="4" fill="4" visible="no" active="no"/>
+<layer number="6" name="Route6" color="1" fill="8" visible="no" active="no"/>
+<layer number="7" name="Route7" color="4" fill="8" visible="no" active="no"/>
+<layer number="8" name="Route8" color="1" fill="2" visible="no" active="no"/>
+<layer number="9" name="Route9" color="4" fill="2" visible="no" active="no"/>
+<layer number="10" name="Route10" color="1" fill="7" visible="no" active="no"/>
+<layer number="11" name="Route11" color="4" fill="7" visible="no" active="no"/>
+<layer number="12" name="Route12" color="1" fill="5" visible="no" active="no"/>
+<layer number="13" name="Route13" color="4" fill="5" visible="no" active="no"/>
+<layer number="14" name="Route14" color="1" fill="6" visible="no" active="no"/>
+<layer number="15" name="Route15" color="4" fill="6" visible="no" active="no"/>
 <layer number="16" name="Bottom" color="1" fill="1" visible="yes" active="yes"/>
 <layer number="17" name="Pads" color="2" fill="1" visible="yes" active="yes"/>
@@
 <attribute name="VERSION" value="1" x="23.5" y="11.2" size="1.778" layer="28" rot="MR90" display="off"/>
 </element>
-<element name="C3" library="rcl" library_urn="urn:adsk.eagle:library:334" package="C0402" value="0.1uF" x="12.27" y="22.69" smashed="yes" rot="MR0">
+<element name="C3" library="rcl" library_urn="urn:adsk.eagle:library:334" package="C0402" value="10uF" x="12.27" y="22.69" smashed="yes" rot="MR0">
 <attribute name="NAME" x="9.595" y="22.675" size="0.635" layer="26" rot="SMR180"/>
 <attribute name="VALUE" x="9.095" y="23.715" size="0.508" layer="28" rot="SMR180"/>
@@
 <attribute name="VALUE" x="19.795" y="17.405" size="0.508" layer="28" rot="SMR270"/>
 </element>
-<element name="C6" library="rcl" library_urn="urn:adsk.eagle:library:334" package="C0402" value="0.1uF" x="19.73" y="25.47" smashed="yes" rot="MR180">
-<attribute name="NAME" x="21.595" y="25.835" size="0.635" layer="26" rot="SMR180"/>
-<attribute name="VALUE" x="21.095" y="26.875" size="0.508" layer="28" rot="SMR180"/>
+<element name="C6" library="rcl" library_urn="urn:adsk.eagle:library:334" package="C0402" value="0.1uF" x="22.23" y="26.47" smashed="yes" rot="MR180">
+<attribute name="NAME" x="24.095" y="26.835" size="0.635" layer="26" rot="SMR180"/>
+<attribute name="VALUE" x="23.595" y="27.875" size="0.508" layer="28" rot="SMR180"/>
 </element>
 <element name="R1" library="rcl" library_urn="urn:adsk.eagle:library:334" package="R0603" value="680" x="17.05" y="27.77" smashed="yes" rot="MR270">
@@
 <attribute name="VALUE" x="18.365" y="13.535" size="0.508" layer="27" rot="SR180"/>
 </element>
-<element name="C8" library="rcl" library_urn="urn:adsk.eagle:library:334" package="C0402" value="?" x="17.21" y="17.27" smashed="yes" rot="MR270">
+<element name="C8" library="rcl" library_urn="urn:adsk.eagle:library:334" package="C0402" value="0.1uF" x="17.21" y="17.27" smashed="yes" rot="MR270">
 <attribute name="NAME" x="17.575" y="15.405" size="0.635" layer="26" rot="SMR270"/>
 <attribute name="VALUE" x="16.115" y="15.905" size="0.508" layer="28" rot="SMR270"/>
 </element>
+<element name="FB2" library="inductors" library_urn="urn:adsk.eagle:library:243" package="0402" value="" x="20" y="25" rot="MR0"/>
 </elements>
 <signals>
@@
 <contactref element="U1" pad="23"/>
 <contactref element="C6" pad="1"/>
-<contactref element="U1" pad="6"/>
-<wire x1="15.13" y1="22.65" x2="12.96" y2="22.65" width="0.254" layer="16"/>
+<wire x1="12.96" y1="22.65" x2="15.13" y2="22.65" width="0.254" layer="16"/>
 <wire x1="12.92" y1="22.69" x2="12.96" y2="22.65" width="0.254" layer="16"/>
 <wire x1="24" y1="14.33" x2="24" y2="12.597" width="0.254" layer="16"/>
@@
 <wire x1="24" y1="14.513025" x2="24.8302" y2="15.343225" width="0.254" layer="16"/>
 <wire x1="24.8302" y1="15.343225" x2="24.8302" y2="22.7498" width="0.254" layer="16"/>
-<wire x1="14.685525" y1="28.7592" x2="15.314475" y2="28.7592" width="0.254" layer="16"/>
-<wire x1="13.2408" y1="27.314475" x2="14.685525" y2="28.7592" width="0.254" layer="16"/>
-<wire x1="12.92" y1="22.69" x2="13.2408" y2="23.0108" width="0.254" layer="16"/>
-<wire x1="13.2408" y1="23.0108" x2="13.2408" y2="27.314475" width="0.254" layer="16"/>
-<wire x1="16.323475" y1="27.7502" x2="17.736775" y2="27.7502" width="0.254" layer="16"/>
-<wire x1="15.314475" y1="28.7592" x2="16.323475" y2="27.7502" width="0.254" layer="16"/>
-<wire x1="24.8302" y1="22.7498" x2="24.2" y2="23.38" width="0.254" layer="16"/>
-<wire x1="24.2" y1="23.38" x2="24.2" y2="23.88" width="0.254" layer="16"/>
-<wire x1="24.2" y1="23.88" x2="22.61" y2="25.47" width="0.254" layer="16"/>
-<wire x1="20.866775" y1="24.6898" x2="19.893225" y2="24.6898" width="0.254" layer="16"/>
-<wire x1="22.61" y1="25.47" x2="21.646975" y2="25.47" width="0.254" layer="16"/>
-<wire x1="19.08" y1="25.47" x2="19.113025" y2="25.47" width="0.254" layer="16"/>
-<wire x1="21.646975" y1="25.47" x2="20.866775" y2="24.6898" width="0.254" layer="16"/>
-<wire x1="19.893225" y1="24.6898" x2="19.113025" y2="25.47" width="0.254" layer="16"/>
-<wire x1="19.08" y1="25.47" x2="18.38" y2="24.77" width="0.254" layer="16"/>
-<wire x1="18.38" y1="24.77" x2="18.38" y2="23.9" width="0.254" layer="16"/>
-<wire x1="17.736775" y1="27.7502" x2="19.08" y2="26.406975" width="0.254" layer="16"/>
-<wire x1="19.08" y1="26.406975" x2="19.08" y2="25.47" width="0.254" layer="16"/>
+<wire x1="24.2" y1="23.38" x2="24.8302" y2="22.7498" width="0.254" layer="16"/>
+<wire x1="24.2" y1="23.88" x2="24.2" y2="23.38" width="0.254" layer="16"/>
 <wire x1="18.38" y1="17.93" x2="18.39" y2="17.92" width="0.254" layer="16"/>
 <wire x1="18.38" y1="17.93" x2="18.38" y2="19.9" width="0.254" layer="16"/>
@@
 <wire x1="11.7408" y1="17.685525" x2="11.7408" y2="20.314475" width="0.254" layer="16"/>
 <wire x1="11.7408" y1="20.314475" x2="12.92" y2="21.493675" width="0.254" layer="16"/>
+<contactref element="FB2" pad="1"/>
+<wire x1="20.65" y1="25" x2="20.65" y2="25.54" width="0.254" layer="16"/>
+<wire x1="20.65" y1="25.54" x2="21.58" y2="26.47" width="0.254" layer="16"/>
+<wire x1="21.58" y1="26.47" x2="20.5852125" y2="26.47" width="0.254" layer="16"/>
+<wire x1="20.5852125" y1="26.47" x2="20.3442125" y2="26.229" width="0.254" layer="16"/>
+<wire x1="15.314475" y1="28.7592" x2="14.685525" y2="28.7592" width="0.254" layer="16"/>
+<wire x1="14.685525" y1="28.7592" x2="13.2408" y2="27.314475" width="0.254" layer="16"/>
+<wire x1="13.2408" y1="23.0108" x2="12.92" y2="22.69" width="0.254" layer="16"/>
+<wire x1="13.2408" y1="27.314475" x2="13.2408" y2="23.0108" width="0.254" layer="16"/>
+<wire x1="17.736775" y1="27.7502" x2="16.323475" y2="27.7502" width="0.254" layer="16"/>
+<wire x1="20.3442125" y1="26.229" x2="19.257975" y2="26.229" width="0.254" layer="16"/>
+<wire x1="19.257975" y1="26.229" x2="17.736775" y2="27.7502" width="0.254" layer="16"/>
+<wire x1="16.323475" y1="27.7502" x2="15.314475" y2="28.7592" width="0.254" layer="16"/>
+<wire x1="21.58" y1="26.47" x2="21.61" y2="26.47" width="0.254" layer="16"/>
+<wire x1="21.61" y1="26.47" x2="24.2" y2="23.88" width="0.254" layer="16"/>
 </signal>
 <signal name="VDD18">
@@
 <wire x1="21.6" y1="15.6" x2="21.6" y2="16.56" width="0.254" layer="1"/>
 </signal>
+<signal name="AVDD">
+<contactref element="U1" pad="6"/>
+<contactref element="FB2" pad="2"/>
+<wire x1="18.38" y1="23.9" x2="18.38" y2="24.38" width="0.254" layer="16"/>
+<wire x1="18.38" y1="24.38" x2="19" y2="25" width="0.254" layer="16"/>
+<wire x1="19" y1="25" x2="19.35" y2="25" width="0.254" layer="16"/>
+</signal>
 </signals>
